Commit message: feat: Implement Raibert controller for spined dog simulation
- Added `main_robot_raibert.py` to integrate the Raibert controller with the MuJoCo simulation.
- Enhanced `MuJoCoSimulation` class with custom control logic for legged locomotion.
- Updated `main_spine.py` to use relative paths for model and URDF files.
- Modified `SpineImpedanceController` to support geometric constraints with soft barrier forces.
- Introduced methods for calculating foot contact forces in `MuJoCoInterface`.
- Adjusted gains and desired positions in the spine controller for improved performance.

File: mujoco_simulation/asset/spine.urdf (robot description, URDF)
Before this commit: robot spine, 4 links, 3 joints
Links:
- added link spine_end_effector, mass 0.001
Joints:
- added joint joint_spine_ee: type fixed, parent front_body, child spine_end_effector, origin xyz=0.00454141 0 0 rpy=0 0 0

File: mujoco_simulation/asset/spined_dog_spine_dyn.urdf (robot description, URDF)
Before this commit: robot spine, 4 links, 3 joints
Links:
- added link spine_end_effector, mass 0.001
Joints:
- added joint joint_spine_ee: type fixed, parent front_body, child spine_end_effector, origin xyz=0.107249862 0 0 rpy=0 0 0
